File: embedded/robot/hardware/expansion_board/expansion_board.brd (EAGLE design)
At the start: 53.3 x 50.2 mm, 50 parts, among them IC1 LM2937, U1 PCA9548APWR, U2 PCA9685PW, U3 MAG3110

Commit message: some boards changes
Parts:
- removed C16: 22uF, resistor:153CLV-0505
- added D1: (no value), adafruit:SOD-523
- added Q1: BSS123, transistor-small-signal:SOT23
- added R7: 50R, resistor:M0805
- added R8: 47k, resistor:M0805
- added U$4: OLED_DISPLAY_096_INCH, my_parts:OLED_DISPLAY_096_INCH
- moved C2 12.5 mm to (21.7, 39.0), turned to 90 degrees
- moved C1 4.76 mm to (21.9, 30.9), turned to 90 degrees
- moved R2 3.05 mm to (22.6, 24.8), turned to 0 degrees
- moved R3 0.45 mm to (27.0, 24.4)
Connections:
- removed net N$17: C16.-, U$3.P$2
- new net N$20: D1.A, R7.2, U$3.P$2
- net +3V3: now also D1.K, U$3.P$1, U$4.P$2
- net GND: now also Q1.2, R8.1, U$4.P$1
- net N$18: now also Q1.1, R8.2; no longer C16.+
- net N$19: now also Q1.3, R7.1; no longer U$3.P$1, U2.16
- net SCL: now also U$4.P$3
- net SDA: now also U$4.P$4
Routing:
- net GND: track 344.8 -> 363.0 mm
- net +3V3: track 238.7 -> 255.7 mm
- net N$18: track 24.0 -> 12.8 mm
- net N$1: track 8.14 -> 16.8 mm
- net AGND: track 8.37 -> 0.00 mm, vias 9 -> 6
- net N$20: track 0.00 -> 8.30 mm
- net N$17: track 8.11 -> 0.00 mm
- net N$19: track 9.20 -> 2.87 mm, vias 1 -> 0
- net SCL: track 126.6 -> 132.4 mm, vias 7 -> 8
- net SDA: track 127.8 -> 128.5 mm

Commit message: expansion board
Parts:
- removed D1: (no value), adafruit:SOD-523
- added D2: (no value), adafruit:SOD-123FL
- added R10, R11, R9: 330, resistor:M0805
- added U$10, U$11, U$12, U$5, U$6, U$7, U$8, U$9: FIDUCIAL, adafruit:FIDUCIAL_1MM
- added U$13: 5MMRGBLED, adafruit:LED5MMRGB
- R7: value 50R -> 22R
- moved Q1 12.8 mm to (30.5, 11.4)
- moved R8 12.2 mm to (29.9, 14.2)
- moved R7 7.91 mm to (27.8, 10.2), turned to 270 degrees
- moved H1 2.84 mm to (36.2, 43.3)
- moved H2 2.84 mm to (16.9, 43.3)
- renumbered SV1 to LEFT, SV2 to FRONT, SV3 to RIGHT, SV4 to REAR, X1 to POWER
Connections:
- new net N$17: R9.2, U$13.1
- new net N$21: R11.2, U$13.4
- new net N$22: R10.2, U$13.2
- new net N$24: R9.1, U2.15
- new net N$25: R10.1, U2.16
- new net N$26: R11.1, U2.17
- net +3V3: now also D2.C; no longer D1.K
- net GND: now also U$13.3
- net N$20: now also D2.A; no longer D1.A
Routing:
- net GND: track 363.0 -> 427.5 mm, vias 28 -> 27
- net N$24: track 0.00 -> 31.7 mm, vias 0 -> 3
- net N$18: track 12.8 -> 26.2 mm
- net N$25: track 0.00 -> 12.5 mm, vias 0 -> 1
- net N$26: track 0.00 -> 11.7 mm, vias 0 -> 1
- net +3V3: track 255.7 -> 248.5 mm
- net SCL_1: track 32.0 -> 26.8 mm
- net SDA_1: track 31.6 -> 27.3 mm
- net N$22: track 0.00 -> 4.26 mm
- net N$17: track 0.00 -> 2.84 mm
- net N$21: track 0.00 -> 2.46 mm
- net N$20: track 8.30 -> 8.80 mm
Other:
- board text added: "+"
