File: embedded/robot/hardware/expansion_board/expansion_board.sch (EAGLE design)
At the start: 50 parts, among them IC1 LM2937, U1 PCA9548APWR, U2 PCA9685PW, U3 MAG3110

Commit message: some boards changes
Parts:
- removed C16: 22uF, resistor:CPOL-EU153CLV-0505
- added D1: (no value), adafruit:DIODESOD-523
- added Q1: BSS123, transistor-small-signal:BSS123
- added R7: 50R, resistor:R-EU_M0805
- added R8: 47k, resistor:R-EU_M0805
- added U$4: OLED_DISPLAY_096_INCH, my_parts:OLED_DISPLAY_096_INCH
Connections:
- removed net N$17: C16.-, U$3.+
- new net N$20: D1.A, R7.2, U$3.+
- net +3V3: now also D1.C, U$3.-, U$4.VCC
- net GND: now also Q1.S, R8.1, U$4.GND
- net N$18: now also Q1.G, R8.2; no longer C16.+
- net N$19: now also Q1.D, R7.1; no longer U$3.-, U2.LED9
- net SCL: now also U$4.SCL
- net SDA: now also U$4.SDA
Changed lines of the file:
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@@
 <layer number="54" name="bGND_GNDA" color="1" fill="9" visible="no" active="no"/>
 <layer number="56" name="wert" color="7" fill="1" visible="no" active="no"/>
+<layer number="57" name="tCAD" color="7" fill="1" visible="no" active="no"/>
 <layer number="91" name="Nets" color="2" fill="1" visible="yes" active="yes"/>
 <layer number="92" name="Busses" color="1" fill="1" visible="yes" active="yes"/>
@@
 <layer number="109" name="ref-old" color="11" fill="1" visible="yes" active="yes"/>
 <layer number="110" name="fp0" color="7" fill="1" visible="yes" active="yes"/>
+<layer number="111" name="LPC17xx" color="7" fill="1" visible="yes" active="yes"/>
+<layer number="112" name="tSilk" color="7" fill="1" visible="yes" active="yes"/>
 <layer number="116" name="Patch_BOT" color="9" fill="4" visible="yes" active="yes"/>
 <layer number="121" name="_tsilk" color="7" fill="1" visible="yes" active="yes"/>
@@
 <layer number="124" name="bTestmark" color="7" fill="1" visible="yes" active="yes"/>
 <layer number="125" name="_tNames" color="7" fill="1" visible="no" active="yes"/>
+<layer number="126" name="_bNames" color="7" fill="1" visible="yes" active="yes"/>
+<layer number="127" name="_tValues" color="7" fill="1" visible="yes" active="yes"/>
+<layer number="128" name="_bValues" color="7" fill="1" visible="yes" active="yes"/>
 <layer number="131" name="prix" color="7" fill="1" visible="yes" active="yes"/>
 <layer number="132" name="test" color="7" fill="1" visible="yes" active="yes"/>
 <layer number="144" name="Drill_legend" color="7" fill="1" visible="yes" active="yes"/>
+<layer number="150" name="Notes" color="7" fill="1" visible="no" active="yes"/>
 <layer number="151" name="HeatSink" color="7" fill="1" visible="yes" active="yes"/>
+<layer number="152" name="_bDocu" color="7" fill="1" visible="yes" active="yes"/>
+<layer number="153" name="FabDoc1" color="6" fill="1" visible="no" active="no"/>
+<layer number="154" name="FabDoc2" color="2" fill="1" visible="no" active="no"/>
+<layer number="155" name="FabDoc3" color="7" fill="15" visible="no" active="no"/>
 <layer number="199" name="Contour" color="7" fill="1" visible="yes" active="yes"/>
 <layer number="200" name="200bmp" color="1" fill="10" visible="yes" active="yes"/>
@@
 <layer number="223" name="223bmp" color="24" fill="1" visible="no" active="no"/>
 <layer number="224" name="224bmp" color="25" fill="1" visible="no" active="no"/>
+<layer number="248" name="Housing" color="7" fill="1" visible="yes" active="yes"/>
+<layer number="249" name="Edge" color="7" fill="1" visible="yes" active="yes"/>
 <layer number="250" name="Descript" color="3" fill="1" visible="no" active="no"/>
 <layer number="251" name="SMDround" color="12" fill="11" visible="no" active="no"/>
@@
 <part name="GND24" library="supply1" deviceset="GND" device=""/>
 <part name="U$3" library="my_parts" deviceset="SPEAKER_KAAG15008C" device=""/>
-<part name="C16" library="resistor" deviceset="CPOL-EU" device="153CLV-0505" value="22uF"/>
+<part name="U$4" library="my_parts" deviceset="OLED_DISPLAY_096_INCH" device=""/>
+<part name="GND25" library="supply1" deviceset="GND" device=""/>
+<part name="+3V23" library="supply1" deviceset="+3V3" device=""/>
+<part name="Q1" library="transistor-small-signal" deviceset="BSS123" device=""/>
+<part name="R7" library="resistor" deviceset="R-EU_" device="M0805" value="50R"/>
+<part name="D1" library="adafruit" deviceset="DIODE" device="SOD-523"/>
+<part name="GND29" library="supply1" deviceset="GND" device=""/>
+<part name="R8" library="resistor" deviceset="R-EU_" device="M0805" value="47k"/>
+<part name="GND30" library="supply1" deviceset="GND" device=""/>
+<part name="+3V24" library="supply1" deviceset="+3V3" device=""/>
 </parts>
 <sheets>
@@
 <instance part="+3V22" gate="G$1" x="320.04" y="114.3" rot="R90"/>
 <instance part="GND24" gate="1" x="342.9" y="114.3" rot="R90"/>
-<instance part="U$3" gate="G$1" x="480.06" y="-2.54"/>
-<instance part="C16" gate="G$1" x="457.2" y="0" rot="R90"/>
+<instance part="U$3" gate="G$1" x="480.06" y="0" rot="MR180"/>
+<instance part="U$4" gate="G$1" x="358.14" y="-73.66"/>
+<instance part="GND25" gate="1" x="337.82" y="-60.96" rot="R180"/>
+<instance part="+3V23" gate="G$1" x="330.2" y="-58.42"/>
+<instance part="Q1" gate="G$1" x="467.36" y="-25.4"/>
+<instance part="R7" gate="G$1" x="467.36" y="-12.7" rot="MR90"/>
+<instance part="D1" gate="G$1" x="464.82" y="2.54" rot="R90"/>
+<instance part="GND29" gate="1" x="467.36" y="-45.72"/>
+<instance part="R8" gate="G$1" x="457.2" y="-35.56" rot="MR90"/>
+<instance part="GND30" gate="1" x="457.2" y="-45.72"/>
+<instance part="+3V24" gate="G$1" x="467.36" y="15.24"/>
 </instances>
 <busses>
@@
 <wire x1="340.36" y1="114.3" x2="335.28" y2="114.3" width="0.1524" layer="91"/>
 </segment>
+<segment>
+<pinref part="U$4" gate="G$1" pin="GND"/>
+<pinref part="GND25" gate="1" pin="GND"/>
+<wire x1="342.9" y1="-66.04" x2="337.82" y2="-66.04" width="0.1524" layer="91"/>
+<wire x1="337.82" y1="-66.04" x2="337.82" y2="-63.5" width="0.1524" layer="91"/>
+</segment>
+<segment>
+<pinref part="R8" gate="G$1" pin="1"/>
+<pinref part="GND30" gate="1" pin="GND"/>
+<wire x1="457.2" y1="-43.18" x2="457.2" y2="-40.64" width="0.1524" layer="91"/>
+</segment>
+<segment>
+<pinref part="GND29" gate="1" pin="GND"/>
+<pinref part="Q1" gate="G$1" pin="S"/>
+<wire x1="467.36" y1="-43.18" x2="467.36" y2="-30.48" width="0.1524" layer="91"/>
+</segment>
 </net>
 <net name="+3V3" class="0">
@@
 <wire x1="327.66" y1="114.3" x2="322.58" y2="114.3" width="0.1524" layer="91"/>
 </segment>
+<segment>
+<pinref part="U$4" gate="G$1" pin="VCC"/>
+<pinref part="+3V23" gate="G$1" pin="+3V3"/>
+<wire x1="342.9" y1="-71.12" x2="330.2" y2="-71.12" width="0.1524" layer="91"/>
+<wire x1="330.2" y1="-71.12" x2="330.2" y2="-60.96" width="0.1524" layer="91"/>
+</segment>
+<segment>
+<wire x1="467.36" y1="5.08" x2="467.36" y2="7.62" width="0.1524" layer="91"/>
+<pinref part="D1" gate="G$1" pin="C"/>
+<wire x1="467.36" y1="7.62" x2="464.82" y2="7.62" width="0.1524" layer="91"/>
+<wire x1="464.82" y1="7.62" x2="464.82" y2="5.08" width="0.1524" layer="91"/>
+<pinref part="+3V24" gate="G$1" pin="+3V3"/>
+<wire x1="467.36" y1="12.7" x2="467.36" y2="7.62" width="0.1524" layer="91"/>
+<junction x="467.36" y="7.62"/>
+<pinref part="U$3" gate="G$1" pin="-"/>
+<wire x1="469.9" y1="5.08" x2="467.36" y2="5.08" width="0.1524" layer="91"/>
+</segment>
 </net>
 <net name="SCL" class="0">
@@
 <label x="467.36" y="58.42" size="1.778" layer="95" rot="R180"/>
 </segment>
+<segment>
+<pinref part="U$4" gate="G$1" pin="SCL"/>
+<wire x1="342.9" y1="-76.2" x2="332.74" y2="-76.2" width="0.1524" layer="91"/>
+<label x="330.2" y="-76.2" size="1.778" layer="95" rot="R180"/>
+</segment>
 </net>
 <net name="SDA" class="0">
@@
 <wire x1="513.08" y1="71.12" x2="520.7" y2="71.12" width="0.1524" layer="91"/>
 <label x="523.24" y="71.12" size="1.778" layer="95"/>
+</segment>
+<segment>
+<pinref part="U$4" gate="G$1" pin="SDA"/>
+<wire x1="342.9" y1="-81.28" x2="332.74" y2="-81.28" width="0.1524" layer="91"/>
+<label x="330.2" y="-81.28" size="1.778" layer="95" rot="R180"/>
 </segment>
 </net>
@@
 </segment>
 </net>
-<net name="N$17" class="0">
-<segment>
+<net name="N$18" class="0">
+<segment>
+<pinref part="U2" gate="A" pin="LED6"/>
+<wire x1="345.44" y1="0" x2="457.2" y2="0" width="0.1524" layer="91"/>
+<pinref part="R8" gate="G$1" pin="2"/>
+<wire x1="457.2" y1="-30.48" x2="457.2" y2="-27.94" width="0.1524" layer="91"/>
+<pinref part="Q1" gate="G$1" pin="G"/>
+<wire x1="457.2" y1="-27.94" x2="457.2" y2="0" width="0.1524" layer="91"/>
+<wire x1="462.28" y1="-27.94" x2="457.2" y2="-27.94" width="0.1524" layer="91"/>
+<junction x="457.2" y="-27.94"/>
+</segment>
+</net>
+<net name="N$19" class="0">
+<segment>
+<pinref part="Q1" gate="G$1" pin="D"/>
+<pinref part="R7" gate="G$1" pin="1"/>
+<wire x1="467.36" y1="-20.32" x2="467.36" y2="-17.78" width="0.1524" layer="91"/>
+</segment>
+</net>
+<net name="N$20" class="0">
+<segment>
+<pinref part="R7" gate="G$1" pin="2"/>
+<wire x1="467.36" y1="-2.54" x2="467.36" y2="-7.62" width="0.1524" layer="91"/>
+<pinref part="D1" gate="G$1" pin="A"/>
+<wire x1="467.36" y1="-2.54" x2="464.82" y2="-2.54" width="0.1524" layer="91"/>
+<wire x1="464.82" y1="-2.54" x2="464.82" y2="0" width="0.1524" layer="91"/>
 <pinref part="U$3" gate="G$1" pin="+"/>
-<pinref part="C16" gate="G$1" pin="-"/>
-<wire x1="469.9" y1="0" x2="462.28" y2="0" width="0.1524" layer="91"/>
-</segment>
-</net>
-<net name="N$18" class="0">
-<segment>
-<pinref part="U2" gate="A" pin="LED6"/>
-<pinref part="C16" gate="G$1" pin="+"/>
-<wire x1="345.44" y1="0" x2="454.66" y2="0" width="0.1524" layer="91"/>
-</segment>
-</net>
-<net name="N$19" class="0">
-<segment>
-<pinref part="U$3" gate="G$1" pin="-"/>
-<pinref part="U2" gate="A" pin="LED9"/>
-<wire x1="345.44" y1="-7.62" x2="469.9" y2="-7.62" width="0.1524" layer="91"/>
-</segment>
-</net>
+<wire x1="469.9" y1="-2.54" x2="467.36" y2="-2.54" width="0.1524" layer="91"/>
+<junction x="467.36" y="-2.54"/>
+</segment>
+</net>

Commit message: expansion board
Parts:
- removed D1: (no value), adafruit:DIODESOD-523
- removed SV1, SV2, SV3, SV4: (no value), con-lstb:MA04-1
- removed X1: (no value), con-wago-500:W237-102
- added D2: (no value), adafruit:DIODE_SOD-123FL
- added FRONT, LEFT, REAR, RIGHT: (no value), con-lstb:MA04-1
- added POWER: (no value), con-wago-500:W237-102
- added R10, R11, R9: 330, resistor:R-EU_M0805
- added U$10, U$11, U$12, U$5, U$6, U$7, U$8, U$9: FIDUCIAL, adafruit:FIDUCIAL
- added U$13: 5MMRGBLED, adafruit:5MMRGBLED
- R7: value 50R -> 22R
Connections:
- new net N$17: R9.2, U$13.BLUE
- new net N$21: R11.2, U$13.RED
- new net N$22: R10.2, U$13.GREEN
- new net N$24: R9.1, U2.LED8
- new net N$25: R10.1, U2.LED9
- new net N$26: R11.1, U2.LED10
- net +3V3: now also D2.C, FRONT.4, LEFT.4, REAR.4, RIGHT.4; no longer D1.C, SV1.4, SV2.4, SV3.4, SV4.4
- net GND: now also FRONT.3, LEFT.3, POWER-2.KL, REAR.3, RIGHT.3, U$13.GND; no longer SV1.3, SV2.3, SV3.3, SV4.3, X1-2.KL
- net N$20: now also D2.A; no longer D1.A
- net SCL_0: now also LEFT.2; no longer SV1.2
- net SCL_1: now also FRONT.2; no longer SV2.2
- net SCL_2: now also RIGHT.2; no longer SV3.2
- net SCL_3: now also REAR.2; no longer SV4.2
- net SDA_0: now also LEFT.1; no longer SV1.1
- net SDA_1: now also FRONT.1; no longer SV2.1
- net SDA_2: now also RIGHT.1; no longer SV3.1
- net SDA_3: now also REAR.1; no longer SV4.1
- net VCC: now also POWER-1.KL; no longer X1-1.KL
Other:
- moved on the sheet: ADC, ADDRESS, C1, C10, C13, C14, C15, C2, C3, C4, C5, C6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
