File: embedded/robot/hardware/expansion_board (copy)/expansion_board.brd (EAGLE design)
At the start: 53.3 x 50.2 mm, 71 parts, among them IC1 LM2937, Q1 BSS123, U1 PCA9548APWR, U2 PCA9685PW, U3 MAG3110, U4 APDS-9960

Commit message: expansion board
Parts:
- removed C16: 100n, resistor:C0805
- removed IO1: SHT21, SparkFun-Sensors:SHT2X
- removed R12, R15: 4k7, resistor:M0805
- removed U4: APDS-9960, SparkFun-Sensors:APDS-9960
- moved U$11 0.45 mm to (49.6, 13.4)
- turned U$1 to 315 degrees
Connections:
- removed net N$27: U4.3, U4.4
- removed net SCL_4: R12.1, U1.14, U4.7
- removed net SDA_4: R15.1, U1.13, U4.1
- net +3V3: no longer C16.1, IO1.5, R12.2, R15.2, U4.5, U4.8
- net GND: no longer C16.2, IO1.2, U4.6
- net SCL: no longer IO1.4
- net SDA: no longer IO1.1
Routing:
- net +3V3: track 280.6 -> 248.5 mm, vias 12 -> 9
- net GND: track 451.7 -> 427.5 mm, vias 26 -> 27
- net SCL_4: track 16.0 -> 0.00 mm
- net SDA_4: track 10.9 -> 0.00 mm
- net N$1: track 23.7 -> 16.8 mm
- net SCL: track 130.0 -> 132.2 mm
- net SDA_0: track 58.9 -> 57.6 mm
- net N$27: track 0.97 -> 0.00 mm
- net SDA: track 129.4 -> 128.5 mm
- net SWDIO: track 45.4 -> 44.6 mm
- net SCL_0: track 56.5 -> 55.9 mm
