File: embedded/robot/hardware/expansion_board (copy)/expansion_board.sch (EAGLE design)
At the start: 71 parts, among them IC1 LM2937, Q1 BSS123, U1 PCA9548APWR, U2 PCA9685PW, U3 MAG3110, U4 APDS-9960

Commit message: expansion board
Parts:
- removed C16: 100n, resistor:C-EUC0805
- removed IO1: SHT21, SparkFun-Sensors:SHT21
- removed R12, R15: 4k7, resistor:R-EU_M0805
- removed U4: APDS-9960, SparkFun-Sensors:APDS-9960
Connections:
- removed net N$27: U4.LDR, U4.LEDK
- removed net SCL_4: R12.1, U1.SC4, U4.SCL
- removed net SDA_4: R15.1, U1.SD4, U4.SDA
- net +3V3: no longer C16.1, IO1.VDD, R12.2, R15.2, U4.LEDA, U4.VDD
- net GND: no longer C16.2, IO1.GND, U4.GND
- net SCL: no longer IO1.SCK
- net SDA: no longer IO1.DATA
Changed lines of the file:
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@@
 <part name="R10" library="resistor" deviceset="R-EU_" device="M0805" value="330"/>
 <part name="R11" library="resistor" deviceset="R-EU_" device="M0805" value="330"/>
-<part name="U4" library="SparkFun-Sensors" deviceset="APDS-9960" device=""/>
-<part name="+3V25" library="supply1" deviceset="+3V3" device=""/>
-<part name="GND32" library="supply1" deviceset="GND" device=""/>
-<part name="R12" library="resistor" deviceset="R-EU_" device="M0805" value="4k7"/>
-<part name="R15" library="resistor" deviceset="R-EU_" device="M0805" value="4k7"/>
-<part name="+3V26" library="supply1" deviceset="+3V3" device=""/>
-<part name="+3V27" library="supply1" deviceset="+3V3" device=""/>
-<part name="C16" library="resistor" deviceset="C-EU" device="C0805" value="100n"/>
-<part name="+3V28" library="supply1" deviceset="+3V3" device=""/>
-<part name="GND33" library="supply1" deviceset="GND" device=""/>
-<part name="IO1" library="SparkFun-Sensors" deviceset="SHT21" device=""/>
-<part name="GND34" library="supply1" deviceset="GND" device=""/>
-<part name="+3V29" library="supply1" deviceset="+3V3" device=""/>
 </parts>
 <sheets>
@@
 <instance part="R10" gate="G$1" x="504.19" y="-20.32" rot="MR90"/>
 <instance part="R11" gate="G$1" x="511.81" y="-20.32" rot="MR90"/>
-<instance part="U4" gate="G$1" x="510.54" y="109.22"/>
-<instance part="+3V25" gate="G$1" x="495.3" y="121.92"/>
-<instance part="GND32" gate="1" x="487.68" y="109.22" rot="R270"/>
-<instance part="R12" gate="G$1" x="529.59" y="115.57" rot="MR90"/>
-<instance part="R15" gate="G$1" x="535.94" y="115.57" rot="MR90"/>
-<instance part="+3V26" gate="G$1" x="529.59" y="123.19"/>
-<instance part="+3V27" gate="G$1" x="535.94" y="123.19"/>
-<instance part="C16" gate="G$1" x="509.27" y="91.44" rot="R90"/>
-<instance part="+3V28" gate="G$1" x="501.65" y="91.44" rot="R90"/>
-<instance part="GND33" gate="1" x="520.7" y="91.44" rot="R90"/>
-<instance part="IO1" gate="G$1" x="528.32" y="45.72" rot="MR180"/>
-<instance part="GND34" gate="1" x="518.16" y="35.56"/>
-<instance part="+3V29" gate="G$1" x="518.16" y="53.34"/>
 </instances>
 <busses>
@@
 <wire x1="508" y1="-17.78" x2="508" y2="-15.24" width="0.1524" layer="91"/>
 </segment>
-<segment>
-<pinref part="U4" gate="G$1" pin="GND"/>
-<pinref part="GND32" gate="1" pin="GND"/>
-<wire x1="497.84" y1="109.22" x2="490.22" y2="109.22" width="0.1524" layer="91"/>
-</segment>
-<segment>
-<pinref part="C16" gate="G$1" pin="2"/>
-<pinref part="GND33" gate="1" pin="GND"/>
-<wire x1="514.35" y1="91.44" x2="518.16" y2="91.44" width="0.1524" layer="91"/>
-</segment>
-<segment>
-<pinref part="IO1" gate="G$1" pin="GND"/>
-<pinref part="GND34" gate="1" pin="GND"/>
-<wire x1="520.7" y1="40.64" x2="518.16" y2="40.64" width="0.1524" layer="91"/>
-<wire x1="518.16" y1="40.64" x2="518.16" y2="38.1" width="0.1524" layer="91"/>
-</segment>
 </net>
 <net name="+3V3" class="0">
@@
 <pinref part="D2" gate="G$1" pin="C"/>
 </segment>
-<segment>
-<pinref part="U4" gate="G$1" pin="VDD"/>
-<pinref part="+3V25" gate="G$1" pin="+3V3"/>
-<wire x1="497.84" y1="114.3" x2="495.3" y2="114.3" width="0.1524" layer="91"/>
-<wire x1="495.3" y1="114.3" x2="495.3" y2="119.38" width="0.1524" layer="91"/>
-<pinref part="U4" gate="G$1" pin="LEDA"/>
-<wire x1="497.84" y1="104.14" x2="495.3" y2="104.14" width="0.1524" layer="91"/>
-<wire x1="495.3" y1="104.14" x2="495.3" y2="114.3" width="0.1524" layer="91"/>
-<junction x="495.3" y="114.3"/>
-</segment>
-<segment>
-<pinref part="R12" gate="G$1" pin="2"/>
-<pinref part="+3V26" gate="G$1" pin="+3V3"/>
-</segment>
-<segment>
-<pinref part="R15" gate="G$1" pin="2"/>
-<pinref part="+3V27" gate="G$1" pin="+3V3"/>
-</segment>
-<segment>
-<pinref part="+3V28" gate="G$1" pin="+3V3"/>
-<pinref part="C16" gate="G$1" pin="1"/>
-<wire x1="506.73" y1="91.44" x2="504.19" y2="91.44" width="0.1524" layer="91"/>
-</segment>
-<segment>
-<pinref part="IO1" gate="G$1" pin="VDD"/>
-<wire x1="520.7" y1="48.26" x2="518.16" y2="48.26" width="0.1524" layer="91"/>
-<wire x1="518.16" y1="48.26" x2="518.16" y2="50.8" width="0.1524" layer="91"/>
-<pinref part="+3V29" gate="G$1" pin="+3V3"/>
-</segment>
 </net>
 <net name="SCL" class="0">
@@
 <label x="292.1" y="58.42" size="1.778" layer="95" rot="R180"/>
 </segment>
-<segment>
-<pinref part="IO1" gate="G$1" pin="SCK"/>
-<wire x1="520.7" y1="45.72" x2="513.08" y2="45.72" width="0.1524" layer="91"/>
-<label x="510.54" y="45.72" size="1.778" layer="95" rot="R180"/>
-</segment>
 </net>
 <net name="SDA" class="0">
@@
 <wire x1="304.8" y1="53.34" x2="294.64" y2="53.34" width="0.1524" layer="91"/>
 <label x="292.1" y="53.34" size="1.778" layer="95" rot="R180"/>
-</segment>
-<segment>
-<pinref part="IO1" gate="G$1" pin="DATA"/>
-<wire x1="520.7" y1="43.18" x2="513.08" y2="43.18" width="0.1524" layer="91"/>
-<label x="510.54" y="43.18" size="1.778" layer="95" rot="R180"/>
 </segment>
 </net>
@@
 </segment>
 </net>
-<net name="N$27" class="0">
-<segment>
-<pinref part="U4" gate="G$1" pin="LEDK"/>
-<wire x1="523.24" y1="114.3" x2="525.78" y2="114.3" width="0.1524" layer="91"/>
-<wire x1="525.78" y1="114.3" x2="525.78" y2="111.76" width="0.1524" layer="91"/>
-<pinref part="U4" gate="G$1" pin="LDR"/>
-<wire x1="525.78" y1="111.76" x2="523.24" y2="111.76" width="0.1524" layer="91"/>
-</segment>
-</net>
-<net name="SCL_4" class="0">
-<segment>
-<pinref part="U1" gate="A" pin="SC4"/>
-<wire x1="264.16" y1="-22.86" x2="254" y2="-22.86" width="0.1524" layer="91"/>
-<label x="251.46" y="-22.86" size="1.778" layer="95" rot="R180"/>
-</segment>
-<segment>
-<pinref part="U4" gate="G$1" pin="SCL"/>
-<wire x1="523.24" y1="106.68" x2="529.59" y2="106.68" width="0.1524" layer="91"/>
-<label x="542.29" y="106.68" size="1.778" layer="95"/>
-<pinref part="R12" gate="G$1" pin="1"/>
-<wire x1="529.59" y1="106.68" x2="539.75" y2="106.68" width="0.1524" layer="91"/>
-<wire x1="529.59" y1="110.49" x2="529.59" y2="106.68" width="0.1524" layer="91"/>
-<junction x="529.59" y="106.68"/>
-</segment>
-</net>
-<net name="SDA_4" class="0">
-<segment>
-<pinref part="U1" gate="A" pin="SD4"/>
-<wire x1="299.72" y1="-5.08" x2="312.42" y2="-5.08" width="0.1524" layer="91"/>
-<label x="314.96" y="-5.08" size="1.778" layer="95"/>
-</segment>
-<segment>
-<pinref part="U4" gate="G$1" pin="SDA"/>
-<wire x1="523.24" y1="104.14" x2="535.94" y2="104.14" width="0.1524" layer="91"/>
-<label x="542.29" y="104.14" size="1.778" layer="95"/>
-<pinref part="R15" gate="G$1" pin="1"/>
-<wire x1="535.94" y1="104.14" x2="539.75" y2="104.14" width="0.1524" layer="91"/>
-<wire x1="535.94" y1="110.49" x2="535.94" y2="104.14" width="0.1524" layer="91"/>
-<junction x="535.94" y="104.14"/>
-</segment>
-</net>
