File: embedded/robot/hardware/main_board_rev_3/main.sch (EAGLE design)
At the start: 90 parts, among them IC1 MAX1555, Q1 8MHz, U1 DRV8830DGQR, U2 STM32F103C6T6A, U3 LSM9DS0, U4 DRV8830DGQR, U5 LM3671MF-3.3, X1 MINI-USB-SCHIELD-32005-201

Commit message: expansion board
Parts:
- renumbered U2 to U2-STM32F303
